File: buck_converter.kicad_sch (KiCad schematic)
At the start: 38 parts, among them U10 MAX5400, U6 TPS54202DDC, U7 TPS54202DDC, U8 MAX5400, U9 TPS54202DDC

Commit message: WIP PCB Routing
Parts:
- L1, L2, L3: footprint Inductor_SMD:L_6.3x6.3_H3 -> Inductor_SMD:L_Bourns_SRN6045TA
Changed lines of the file:
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@@
     (property "Reference" "L2" (id 0) (at 114.3 60.96 90))
     (property "Value" "22uH 3A" (id 1) (at 114.3 63.5 90))
-    (property "Footprint" "Inductor_SMD:L_6.3x6.3_H3" (id 2) (at 114.3 67.31 0)
+    (property "Footprint" "Inductor_SMD:L_Bourns_SRN6045TA" (id 2) (at 114.3 67.31 0)
       (effects (font (size 1.27 1.27)) hide)
     )
@@
     (property "Reference" "L3" (id 0) (at 114.3 128.27 90))
     (property "Value" "22uH 3A" (id 1) (at 114.3 130.81 90))
-    (property "Footprint" "Inductor_SMD:L_6.3x6.3_H3" (id 2) (at 114.3 134.62 0)
+    (property "Footprint" "Inductor_SMD:L_Bourns_SRN6045TA" (id 2) (at 114.3 134.62 0)
       (effects (font (size 1.27 1.27)) hide)
     )
@@
     (property "Reference" "L1" (id 0) (at 114.3 25.4 90))
     (property "Value" "22uH 3A" (id 1) (at 114.3 27.94 90))
-    (property "Footprint" "Inductor_SMD:L_6.3x6.3_H3" (id 2) (at 114.3 31.75 0)
-      (effects (font (size 1.27 1.27)) hide)
-    )
+    (property "Footprint" "Inductor_SMD:L_Bourns_SRN6045TA" (id 2) (at 114.3 31.75 0)
+      (effects (font (size 1.27 1.27)) hide)
+    )

Commit message: Power optimization, add Aisler Assembly MPN info
Parts:
- C10, C13, C14, C16, C19, C20, C23, C26, C27: MPN (none) -> 22uF 25V X7R
- C11, C15, C17, C21, C22, C24, C28, C9: MPN (none) -> 100nF 50V X7R
- C12, C18, C25: MPN (none) -> 56pF 50V C0G
- L1, L2, L3: MPN (none) -> SRN6045TA-220M
- R28, R30, R31, R34, R35: MPN (none) -> 100K 1%
- R29: MPN (none) -> 22K 1%
- R32, R36: value 3K3 -> 2K4; MPN (none) -> 2K4 1%
- R33, R37: value 680R -> 220R; MPN (none) -> 220R 1%
- U10, U8: MPN (none) -> MAX5400EKA+T
- U6, U7, U9: MPN (none) -> TPS54202DDCR
Other:
- note added: "Vout(min) = 1.8V Vout(max) = 23.3V"
- note removed: "Vout(min) = 1.8V Vout(max) = 15.5V"
Changed lines of the file:
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@@
     (stroke (width 0) (type default) (color 0 0 0 0))
   )
-  (text "Vout(min) = 1.8V\nVout(max) = 15.5V" (at 130.81 154.94 0)
+  (text "Vout(min) = 1.8V\nVout(max) = 23.3V" (at 130.81 154.94 0)
     (effects (font (size 1.27 1.27)) (justify left bottom))
   )
@@
     (effects (font (size 1.27 1.27)) (justify left bottom))
   )
-  (text "Vout(min) = 1.8V\nVout(max) = 15.5V" (at 130.81 87.63 0)
+  (text "Vout(min) = 1.8V\nVout(max) = 23.3V" (at 130.81 87.63 0)
     (effects (font (size 1.27 1.27)) (justify left bottom))
   )
@@
       (effects (font (size 1.27 1.27)) (justify left))
     )
-    (property "Value" "3K3" (id 1) (at 121.92 81.2799 0)
+    (property "Value" "2K4" (id 1) (at 121.92 81.2799 0)
       (effects (font (size 1.27 1.27)) (justify left))
     )
@@
     )
     (property "Datasheet" "~" (id 3) (at 119.38 80.01 0)
+      (effects (font (size 1.27 1.27)) hide)
+    )
+    (property "MPN" "2K4 1%" (id 4) (at 119.38 80.01 0)
       (effects (font (size 1.27 1.27)) hide)
     )
@@
       (effects (font (size 1.27 1.27)) hide)
     )
+    (property "MPN" "TPS54202DDCR" (id 4) (at 90.17 69.85 0)
+      (effects (font (size 1.27 1.27)) hide)
+    )
     (pin "1")
     (pin "2")
@@
       (effects (font (size 1.27 1.27)) hide)
     )
+    (property "MPN" "100nF 50V X7R" (id 4) (at 106.68 154.94 0)
+      (effects (font (size 1.27 1.27)) hide)
+    )
     (pin "1")
     (pin "2")
@@
     )
     (property "Datasheet" "~" (id 3) (at 106.68 87.63 0)
+      (effects (font (size 1.27 1.27)) hide)
+    )
+    (property "MPN" "100nF 50V X7R" (id 4) (at 106.68 87.63 0)
       (effects (font (size 1.27 1.27)) hide)
     )
@@
       (effects (font (size 1.27 1.27)) (justify left))
     )
-    (property "Value" "3K3" (id 1) (at 121.92 148.5899 0)
+    (property "Value" "2K4" (id 1) (at 121.92 148.5899 0)
       (effects (font (size 1.27 1.27)) (justify left))
     )
@@
     )
     (property "Datasheet" "~" (id 3) (at 119.38 147.32 0)
+      (effects (font (size 1.27 1.27)) hide)
+    )
+    (property "MPN" "2K4 1%" (id 4) (at 119.38 147.32 0)
       (effects (font (size 1.27 1.27)) hide)
     )
@@
       (effects (font (size 1.27 1.27)) hide)
     )
+    (property "MPN" "100K 1%" (id 4) (at 119.38 35.56 0)
+      (effects (font (size 1.27 1.27)) hide)
+    )
     (pin "1")
     (pin "2")
@@
     )
     (property "Datasheet" "https://datasheet.lcsc.com/lcsc/2105241240_Maxim-Integrated-MAX5400EKA-T_C516784.pdf" (id 3) (at 139.7 184.15 0)
+      (effects (font (size 1.27 1.27)) hide)
+    )
+    (property "MPN" "MAX5400EKA+T" (id 4) (at 90.17 168.91 0)
       (effects (font (size 1.27 1.27)) hide)
     )
@@
       (effects (font (size 1.27 1.27)) hide)
     )
+    (property "MPN" "22uF 25V X7R" (id 4) (at 139.7 71.12 0)
+      (effects (font (size 1.27 1.27)) hide)
+    )
     (pin "1")
     (pin "2")
@@
       (effects (font (size 1.27 1.27)) hide)
     )
+    (property "MPN" "SRN6045TA-220M" (id 4) (at 114.3 67.31 0)
+      (effects (font (size 1.27 1.27)) hide)
+    )
     (pin "1")
     (pin "2")
@@
     )
     (property "Datasheet" "~" (id 3) (at 149.86 138.43 0)
+      (effects (font (size 1.27 1.27)) hide)
+    )
+    (property "MPN" "22uF 25V X7R" (id 4) (at 149.86 138.43 0)
       (effects (font (size 1.27 1.27)) hide)
     )
@@
       (effects (font (size 1.27 1.27)) hide)
     )
+    (property "MPN" "100nF 50V X7R" (id 4) (at 105.41 31.75 0)
+      (effects (font (size 1.27 1.27)) hide)
+    )
     (pin "1")
     (pin "2")
@@
     )
     (property "Datasheet" "~" (id 3) (at 119.38 71.12 0)
+      (effects (font (size 1.27 1.27)) hide)
+    )
+    (property "MPN" "100K 1%" (id 4) (at 119.38 71.12 0)
       (effects (font (size 1.27 1.27)) hide)
     )
@@
       (effects (font (size 1.27 1.27)) hide)
     )
+    (property "MPN" "100nF 50V X7R" (id 4) (at 105.41 134.62 0)
+      (effects (font (size 1.27 1.27)) hide)
+    )
     (pin "1")
     (pin "2")
@@
       (effects (font (size 1.27 1.27)) hide)
     )
+    (property "MPN" "SRN6045TA-220M" (id 4) (at 114.3 134.62 0)
+      (effects (font (size 1.27 1.27)) hide)
+    )
     (pin "1")
     (pin "2")
@@
     )
     (property "Datasheet" "~" (id 3) (at 72.39 76.2 0)
+      (effects (font (size 1.27 1.27)) hide)
+    )
+    (property "MPN" "100K 1%" (id 4) (at 72.39 76.2 0)
       (effects (font (size 1.27 1.27)) hide)
     )
@@
       (effects (font (size 1.27 1.27)) hide)
     )
+    (property "MPN" "56pF 50V C0G" (id 4) (at 129.54 138.43 0)
+      (effects (font (size 1.27 1.27)) hide)
+    )
     (pin "1")
     (pin "2")
@@
     )
     (property "Datasheet" "~" (id 3) (at 149.86 71.12 0)
+      (effects (font (size 1.27 1.27)) hide)
+    )
+    (property "MPN" "22uF 25V X7R" (id 4) (at 149.86 71.12 0)
       (effects (font (size 1.27 1.27)) hide)
     )
@@
       (effects (font (size 1.27 1.27)) hide)
     )
+    (property "MPN" "TPS54202DDCR" (id 4) (at 90.17 34.29 0)
+      (effects (font (size 1.27 1.27)) hide)
+    )
     (pin "1")
     (pin "2")
@@
       (effects (font (size 1.27 1.27)) hide)
     )
+    (property "MPN" "100nF 50V X7R" (id 4) (at 68.58 35.56 0)
+      (effects (font (size 1.27 1.27)) hide)
+    )
     (pin "1")
     (pin "2")
@@
     )
     (property "Datasheet" "~" (id 3) (at 149.86 35.56 0)
+      (effects (font (size 1.27 1.27)) hide)
+    )
+    (property "MPN" "22uF 25V X7R" (id 4) (at 149.86 35.56 0)
       (effects (font (size 1.27 1.27)) hide)
     )
@@
       (effects (font (size 1.27 1.27)) hide)
     )
+    (property "MPN" "TPS54202DDCR" (id 4) (at 90.17 137.16 0)
+      (effects (font (size 1.27 1.27)) hide)
+    )
     (pin "1")
     (pin "2")
@@
       (effects (font (size 1.27 1.27)) hide)
     )
+    (property "MPN" "100K 1%" (id 4) (at 119.38 138.43 0)
+      (effects (font (size 1.27 1.27)) hide)
+    )
     (pin "1")
     (pin "2")
@@
     )
     (property "Datasheet" "https://datasheet.lcsc.com/lcsc/2105241240_Maxim-Integrated-MAX5400EKA-T_C516784.pdf" (id 3) (at 139.7 116.84 0)
+      (effects (font (size 1.27 1.27)) hide)
+    )
+    (property "MPN" "MAX5400EKA+T" (id 4) (at 90.17 101.6 0)
       (effects (font (size 1.27 1.27)) hide)
     )
@@
       (effects (font (size 1.27 1.27)) (justify left))
     )
-    (property "Value" "680R" (id 1) (at 121.92 88.8999 0)
+    (property "Value" "220R" (id 1) (at 121.92 88.8999 0)
       (effects (font (size 1.27 1.27)) (justify left))
     )
@@
     )
     (property "Datasheet" "~" (id 3) (at 119.38 87.63 0)
+      (effects (font (size 1.27 1.27)) hide)
+    )
+    (property "MPN" "220R 1%" (id 4) (at 119.38 87.63 0)
       (effects (font (size 1.27 1.27)) hide)
     )
@@
       (effects (font (size 1.27 1.27)) hide)
     )
+    (property "MPN" "100nF 50V X7R" (id 4) (at 105.41 67.31 0)
+      (effects (font (size 1.27 1.27)) hide)
+    )
     (pin "1")
     (pin "2")
@@
       (effects (font (size 1.27 1.27)) hide)
     )
+    (property "MPN" "100K 1%" (id 4) (at 72.39 143.51 0)
+      (effects (font (size 1.27 1.27)) hide)
+    )
     (pin "1")
     (pin "2")
@@
       (effects (font (size 1.27 1.27)) (justify left))
     )
-    (property "Value" "680R" (id 1) (at 121.92 156.2099 0)
+    (property "Value" "220R" (id 1) (at 121.92 156.2099 0)
       (effects (font (size 1.27 1.27)) (justify left))
     )
@@
     )
     (property "Datasheet" "~" (id 3) (at 119.38 154.94 0)
+      (effects (font (size 1.27 1.27)) hide)
+    )
+    (property "MPN" "220R 1%" (id 4) (at 119.38 154.94 0)
       (effects (font (size 1.27 1.27)) hide)
     )
@@
       (effects (font (size 1.27 1.27)) hide)
     )
+    (property "MPN" "22uF 25V X7R" (id 4) (at 58.42 35.56 0)
+      (effects (font (size 1.27 1.27)) hide)
+    )
     (pin "1")
     (pin "2")
@@
     )
     (property "Datasheet" "~" (id 3) (at 129.54 35.56 0)
+      (effects (font (size 1.27 1.27)) hide)
+    )
+    (property "MPN" "56pF 50V C0G" (id 4) (at 129.54 35.56 0)
       (effects (font (size 1.27 1.27)) hide)
     )
@@
       (effects (font (size 1.27 1.27)) hide)
     )
+    (property "MPN" "22K 1%" (id 4) (at 119.38 44.45 0)
+      (effects (font (size 1.27 1.27)) hide)
+    )
     (pin "1")
     (pin "2")
@@
     )
     (property "Datasheet" "~" (id 3) (at 139.7 138.43 0)
+      (effects (font (size 1.27 1.27)) hide)
+    )
+    (property "MPN" "22uF 25V X7R" (id 4) (at 139.7 138.43 0)
       (effects (font (size 1.27 1.27)) hide)
     )
@@
       (effects (font (size 1.27 1.27)) hide)
     )
+    (property "MPN" "22uF 25V X7R" (id 4) (at 139.7 35.56 0)
+      (effects (font (size 1.27 1.27)) hide)
+    )
     (pin "1")
     (pin "2")
@@
       (effects (font (size 1.27 1.27)) hide)
     )
+    (property "MPN" "56pF 50V C0G" (id 4) (at 129.54 71.12 0)
+      (effects (font (size 1.27 1.27)) hide)
+    )
     (pin "1")
     (pin "2")
@@
       (effects (font (size 1.27 1.27)) hide)
     )
+    (property "MPN" "100nF 50V X7R" (id 4) (at 44.45 71.12 0)
+      (effects (font (size 1.27 1.27)) hide)
+    )
     (pin "1")
     (pin "2")
@@
       (effects (font (size 1.27 1.27)) hide)
     )
+    (property "MPN" "22uF 25V X7R" (id 4) (at 34.29 71.12 0)
+      (effects (font (size 1.27 1.27)) hide)
+    )
     (pin "1")
     (pin "2")
@@
     )
     (property "Datasheet" "~" (id 3) (at 34.29 138.43 0)
+      (effects (font (size 1.27 1.27)) hide)
+    )
+    (property "MPN" "22uF 25V X7R" (id 4) (at 34.29 138.43 0)
       (effects (font (size 1.27 1.27)) hide)
     )
@@
       (effects (font (size 1.27 1.27)) hide)
     )
+    (property "MPN" "SRN6045TA-220M" (id 4) (at 114.3 31.75 0)
+      (effects (font (size 1.27 1.27)) hide)
+    )
     (pin "1")
     (pin "2")
@@
       (effects (font (size 1.27 1.27)) hide)
     )
+    (property "MPN" "100nF 50V X7R" (id 4) (at 44.45 138.43 0)
+      (effects (font (size 1.27 1.27)) hide)
+    )

Commit message: Create IBOM, Add sheet info
Other:
- company: (none) -> Sleepy Pony Labs
- title: (none) -> Dual Rail Breadboard Power Supply
Changed lines of the file:
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@@
 (kicad_sch (version 20211123) (generator eeschema)
   (paper "A4")
+  (title_block
+    (title "Dual Rail Breadboard Power Supply")
+    (date "2023-06-11")
+    (rev "1")
+    (company "Sleepy Pony Labs")
+  )
   (junction (at 129.54 67.31) (diameter 0) (color 0 0 0 0)
   )
