File: microcontroller.kicad_sch (KiCad schematic)
At the start: 18 parts, among them J3 ST-Link, U11 SL6206-33NR, U12 STM32F070RBT6, Y1 8MHz

Commit message: WIP PCb routing
Parts:
- removed C35: 100nF, Capacitor_SMD:C_0603_1608Metric, symbol Device:C_Small
- removed J3: ST-Link, Connector_PinHeader_2.54mm:PinHeader_1x06_P2.54mm_Vertical, symbol Connector:Conn_01x06_Male
- added J3: ST-Link, Connector_PinHeader_1.27mm:PinHeader_2x03_P1.27mm_Vertical_SMD, symbol Connector_Generic:Conn_02x03_Odd_Even
Connections:
- net BTN_ON_LEFT: now also U12.29 (PB10); no longer U12.3 (PC14)
- net BTN_ON_RIGHT: now also U12.25 (PC5); no longer U12.4 (PC15)
- net BTN_SEL_LEFT: now also U12.30 (PB11); no longer U12.52 (PC11)
- net BTN_SEL_MEAS: now also U12.27 (PB1); no longer U12.2 (PC13)
- net BTN_SEL_RIGHT: now also U12.24 (PC4); no longer U12.53 (PC12)
- net BUCK_EN_LEFT: now also U12.40 (PC9); no longer U12.27 (PB1)
- net BUCK_EN_RIGHT: now also U12.3 (PC14); no longer U12.61 (PB8)
- net GND: now also J3.4 (Pin_4)
- net ISENSE_LEFT: now also U12.9 (PC1); no longer U12.14 (PA0)
- net ISENSE_RIGHT: now also U12.16 (PA2); no longer U12.8 (PC0)
- net ISENSE_VIN: now also U12.15 (PA1); no longer U12.11 (PC3)
- net NRST: now also J3.5 (Pin_5)
- net PD_FAULT: now also U12.43 (PA10); no longer U12.26 (PB0)
- net POT_LEFT: now also U12.10 (PC2); no longer U12.16 (PA2)
- net POT_RIGHT: now also U12.11 (PC3); no longer U12.10 (PC2)
- net RELAY_LEFT: now also U12.42 (PA9); no longer U12.28 (PB2)
- net RELAY_RIGHT: now also U12.4 (PC15); no longer U12.62 (PB9)
- net SWCLK: now also J3.3 (Pin_3)
- net SWDIO: now also J3.6 (Pin_6)
- net SWO: now also J3.1 (Pin_1)
- net VSENSE_LEFT: now also U12.8 (PC0); no longer U12.15 (PA1)
- net VSENSE_RIGHT: now also U12.17 (PA3); no longer U12.9 (PC1)
- net VSENSE_VIN: now also U12.14 (PA0); no longer U12.17 (PA3)
- net ~{DP_CS_RIGHT}: now also U12.2 (PC13); no longer U12.42 (PA9)
- net ~{SHDN_LEFT}: now also U12.28 (PB2); no longer U12.20 (PA4)
- net ~{SHDN_RIGHT}: now also U12.26 (PB0); no longer U12.24 (PC4)
- net +3V3 renamed +3.3V
- net +3.3V: now also J3.2 (Pin_2)
- no-connect marks 16 -> 0
Other:
- note removed: "VDD SWCLK GND SWDIO NRST SWO"

Commit message: Power optimization, add Aisler Assembly MPN info
Parts:
- C29, C30, C31, C32, C33, C34, C36: MPN (none) -> 100nF 50V X7R
- C37, C38: MPN (none) -> 1uF 50V X7R
- C39, C40: MPN (none) -> 20pF 50V C0G
- R38, R39: MPN (none) -> 100K 1%
- U11: MPN (none) -> XC6206P332MRN
- U12: MPN (none) -> STM32F070RBT6
- Y1: MPN (none) -> ECS-80-8-30-JGN-TR
Changed lines of the file:
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@@
+      (effects (font (size 1.27 1.27)) hide)
+    )
+    (property "MPN" "100nF 50V X7R" (id 4) (at 86.36 40.64 0)
       (effects (font (size 1.27 1.27)) hide)
     )
@@
     )
     (property "Datasheet" "~" (id 3) (at 74.93 40.64 0)
+      (effects (font (size 1.27 1.27)) hide)
+    )
+    (property "MPN" "100nF 50V X7R" (id 4) (at 74.93 40.64 0)
       (effects (font (size 1.27 1.27)) hide)
     )
@@
     )
     (property "Datasheet" "~" (id 3) (at 63.5 40.64 0)
+      (effects (font (size 1.27 1.27)) hide)
+    )
+    (property "MPN" "100nF 50V X7R" (id 4) (at 63.5 40.64 0)
       (effects (font (size 1.27 1.27)) hide)
     )
@@
       (effects (font (size 1.27 1.27)) hide)
     )
+    (property "MPN" "20pF 50V C0G" (id 4) (at 41.91 99.06 0)
+      (effects (font (size 1.27 1.27)) hide)
+    )
     (pin "1")
     (pin "2")
@@
       (effects (font (size 1.27 1.27)) hide)
     )
+    (property "MPN" "100K 1%" (id 4) (at 59.69 73.66 0)
+      (effects (font (size 1.27 1.27)) hide)
+    )
     (pin "1")
     (pin "2")
@@
       (effects (font (size 1.27 1.27)) hide)
     )
+    (property "MPN" "100nF 50V X7R" (id 4) (at 52.07 40.64 0)
+      (effects (font (size 1.27 1.27)) hide)
+    )
     (pin "1")
     (pin "2")
@@
     )
     (property "Datasheet" "~" (id 3) (at 157.48 81.28 0)
+      (effects (font (size 1.27 1.27)) hide)
+    )
+    (property "MPN" "1uF 50V X7R" (id 4) (at 157.48 81.28 0)
       (effects (font (size 1.27 1.27)) hide)
     )
@@
     )
     (property "Datasheet" "http://www.st.com/st-web-ui/static/active/en/resource/technical/document/datasheet/DM00141386.pdf" (id 3) (at 86.36 104.14 0)
+      (effects (font (size 1.27 1.27)) hide)
+    )
+    (property "MPN" "STM32F070RBT6" (id 4) (at 86.36 104.14 0)
       (effects (font (size 1.27 1.27)) hide)
     )
@@
       (effects (font (size 1.27 1.27)) hide)
     )
+    (property "MPN" "100K 1%" (id 4) (at 48.26 66.04 0)
+      (effects (font (size 1.27 1.27)) hide)
+    )
     (pin "1")
     (pin "2")
@@
     )
     (property "Datasheet" "~" (id 3) (at 54.61 95.25 0)
+      (effects (font (size 1.27 1.27)) hide)
+    )
+    (property "MPN" "ECS-80-8-30-JGN-TR" (id 4) (at 54.61 95.25 0)
       (effects (font (size 1.27 1.27)) hide)
     )
@@
       (effects (font (size 1.27 1.27)) hide)
     )
+    (property "MPN" "XC6206P332MRN" (id 4) (at 171.45 76.2 0)
+      (effects (font (size 1.27 1.27)) hide)
+    )
     (pin "1")
     (pin "2")
@@
     )
     (property "Datasheet" "~" (id 3) (at 109.22 40.64 0)
+      (effects (font (size 1.27 1.27)) hide)
+    )
+    (property "MPN" "100nF 50V X7R" (id 4) (at 109.22 40.64 0)
       (effects (font (size 1.27 1.27)) hide)
     )
@@
       (effects (font (size 1.27 1.27)) hide)
     )
+    (property "MPN" "100nF 50V X7R" (id 4) (at 97.79 40.64 0)
+      (effects (font (size 1.27 1.27)) hide)
+    )
     (pin "1")
     (pin "2")
@@
     )
     (property "Datasheet" "~" (id 3) (at 48.26 73.66 0)
+      (effects (font (size 1.27 1.27)) hide)
+    )
+    (property "MPN" "100nF 50V X7R" (id 4) (at 48.26 73.66 0)
       (effects (font (size 1.27 1.27)) hide)
     )
@@
       (effects (font (size 1.27 1.27)) hide)
     )
+    (property "MPN" "20pF 50V C0G" (id 4) (at 41.91 91.44 0)
+      (effects (font (size 1.27 1.27)) hide)
+    )
     (pin "1")
     (pin "2")
@@
       (effects (font (size 1.27 1.27)) hide)
     )
+    (property "MPN" "1uF 50V X7R" (id 4) (at 182.88 81.28 0)
+      (effects (font (size 1.27 1.27)) hide)
+    )

Commit message: Create IBOM, Add sheet info
Other:
- company: (none) -> Sleepy Pony Labs
- title: (none) -> Dual Rail Breadboard Power Supply
Changed lines of the file:
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@@
 (kicad_sch (version 20211123) (generator eeschema)
   (paper "A4")
+  (title_block
+    (title "Dual Rail Breadboard Power Supply")
+    (date "2023-06-11")
+    (rev "1")
+    (company "Sleepy Pony Labs")
+  )
   (junction (at 86.36 151.13) (diameter 0) (color 0 0 0 0)
   )
