File: user_interface.kicad_sch (KiCad schematic)
At the start: 43 parts, among them J4 SHDN, J5 SHDN, SW1 Button, SW2 Button, SW3 Button, SW4 Button, SW5 Button, U13 GN1640T, U14 74LVC1G14, U15 74LVC1G14

Commit message: Add mounting holes, WIP routing
Parts:
- removed R48, R49, R50, R51, R52: 10K, Resistor_SMD:R_0603_1608Metric, symbol Device:R
- added H1, H2: MountingHole, MountingHole:MountingHole_3.2mm_M3_Pad, symbol Mechanical:MountingHole
Connections:
- net SEG1: now also D10.2 (A); no longer D5.2 (A)
- net SEG2: now also D9.2 (A); no longer D6.2 (A)
- net SEG3: now also D11.2 (A); no longer D7.2 (A)
- net SEG4: now also D6.2 (A); no longer D8.2 (A)
- net SEG5: now also D5.2 (A); no longer D9.2 (A)
- net SEG6: now also D7.2 (A); no longer D10.2 (A)
- net SEG7: now also D12.2 (A); no longer D11.2 (A)
- net SEG8: now also D8.2 (A); no longer D12.2 (A)
- net GR12: now reaches U13.1 (GRID12)
- net GR12: now also LED2.12 (CC1)
- net GR13: now reaches U13.2 (GRID13)
- net GR13: now also LED1.9 (CC2)
- net GR10: now reaches U13.27 (GRID10)
- net GR10: now also D10.1 (K), D11.1 (K), D12.1 (K), D5.1 (K), D6.1 (K), D7.1 (K), D8.1 (K), D9.1 (K)
- net GR11: now reaches U13.28 (GRID11)
- net GR11: now also LED1.12 (CC1)
- net GR14: now reaches U13.3 (GRID14)
- net GR14: now also LED2.9 (CC2)
- net GR15: now reaches U13.4 (GRID15)
- net GR15: now also LED1.8 (CC3)
- net GR16: now reaches U13.5 (GRID16)
- net GR16: now also LED2.8 (CC3)
- net GR1: no longer names the net of U13.18 (GRID1)
- net GR1: no longer LED1.12 (CC1)
- net GR2: no longer names the net of U13.19 (GRID2)
- net GR2: no longer LED1.9 (CC2)
- net GR3: no longer names the net of U13.20 (GRID3)
- net GR3: no longer LED1.8 (CC3)
- net GR4: no longer names the net of U13.21 (GRID4)
- net GR4: no longer LED2.12 (CC1)
- net GR5: no longer names the net of U13.22 (GRID5)
- net GR5: no longer LED2.9 (CC2)
- net GR6: no longer names the net of U13.23 (GRID6)
- net GR6: no longer LED2.8 (CC3)
- removed net GR7: D10.1 (K), D11.1 (K), D12.1 (K), D5.1 (K), D6.1 (K), D7.1 (K), D8.1 (K), D9.1 (K), U13.24 (GRID7)

Commit message: WIP PCB routing
Parts:
- removed H1, H2: MountingHole, MountingHole:MountingHole_3.2mm_M3_Pad, symbol Mechanical:MountingHole
- added H1, H2: MountingHole_Pad, MountingHole:MountingHole_3.2mm_M3_Pad, symbol Mechanical:MountingHole_Pad
Connections:
- no-connect marks 9 -> 11
Changed lines of the file:
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@@
   (no_connect (at 92.71 54.61))
   (no_connect (at 92.71 46.99))
+  (no_connect (at 254 143.51))
+  (no_connect (at 254 133.35))
   (no_connect (at 92.71 64.77))
   (no_connect (at 92.71 52.07))
@@
     )
     (pin "1")
-  )
-  (symbol (lib_id "Mechanical:MountingHole") (at 256.54 142.24 0) (unit 1)
-    (in_bom yes) (on_board yes) (fields_autoplaced)
-    (property "Reference" "H2" (id 0) (at 259.08 140.9699 0)
-      (effects (font (size 1.27 1.27)) (justify left))
-    )
-    (property "Value" "MountingHole" (id 1) (at 259.08 143.5099 0)
-      (effects (font (size 1.27 1.27)) (justify left))
-    )
-    (property "Footprint" "MountingHole:MountingHole_3.2mm_M3_Pad" (id 2) (at 256.54 142.24 0)
-      (effects (font (size 1.27 1.27)) hide)
-    )
-    (property "Datasheet" "~" (id 3) (at 256.54 142.24 0)
-      (effects (font (size 1.27 1.27)) hide)
-    )
   )
   (symbol (lib_id "Device:R") (at 209.55 44.45 0) (unit 1)
@@
     (pin "9")
   )
+  (symbol (lib_id "Mechanical:MountingHole_Pad") (at 254 130.81 0) (unit 1)
+    (in_bom yes) (on_board yes) (fields_autoplaced)
+    (property "Reference" "H1" (id 0) (at 256.54 128.2699 0)
+      (effects (font (size 1.27 1.27)) (justify left))
+    )
+    (property "Value" "MountingHole_Pad" (id 1) (at 256.54 130.8099 0)
+      (effects (font (size 1.27 1.27)) (justify left))
+    )
+    (property "Footprint" "MountingHole:MountingHole_3.2mm_M3_Pad" (id 2) (at 254 130.81 0)
+      (effects (font (size 1.27 1.27)) hide)
+    )
+    (property "Datasheet" "~" (id 3) (at 254 130.81 0)
+      (effects (font (size 1.27 1.27)) hide)
+    )
+    (pin "1")
+  )
   (symbol (lib_id "breadboard_supply:74LVC1G14") (at 63.5 137.16 0) (unit 1)
     (in_bom yes) (on_board yes)
@@
     (pin "2")
   )
+  (symbol (lib_id "Mechanical:MountingHole_Pad") (at 254 140.97 0) (unit 1)
+    (in_bom yes) (on_board yes) (fields_autoplaced)
+    (property "Reference" "H2" (id 0) (at 256.54 138.4299 0)
+      (effects (font (size 1.27 1.27)) (justify left))
+    )
+    (property "Value" "MountingHole_Pad" (id 1) (at 256.54 140.9699 0)
+      (effects (font (size 1.27 1.27)) (justify left))
+    )
+    (property "Footprint" "MountingHole:MountingHole_3.2mm_M3_Pad" (id 2) (at 254 140.97 0)
+      (effects (font (size 1.27 1.27)) hide)
+    )
+    (property "Datasheet" "~" (id 3) (at 254 140.97 0)
+      (effects (font (size 1.27 1.27)) hide)
+    )
+    (pin "1")
+  )
   (symbol (lib_id "Device:LED") (at 137.16 156.21 0) (mirror y) (unit 1)
     (in_bom yes) (on_board yes)
@@
     (pin "2")
   )
-  (symbol (lib_id "Mechanical:MountingHole") (at 256.54 135.89 0) (unit 1)
-    (in_bom yes) (on_board yes) (fields_autoplaced)
-    (property "Reference" "H1" (id 0) (at 259.08 134.6199 0)
-      (effects (font (size 1.27 1.27)) (justify left))
-    )
-    (property "Value" "MountingHole" (id 1) (at 259.08 137.1599 0)
-      (effects (font (size 1.27 1.27)) (justify left))
-    )
-    (property "Footprint" "MountingHole:MountingHole_3.2mm_M3_Pad" (id 2) (at 256.54 135.89 0)
-      (effects (font (size 1.27 1.27)) hide)
-    )
-    (property "Datasheet" "~" (id 3) (at 256.54 135.89 0)
-      (effects (font (size 1.27 1.27)) hide)
-    )
-  )
   (symbol (lib_id "Switch:SW_Push") (at 219.71 97.79 0) (unit 1)

Commit message: Power optimization, add Aisler Assembly MPN info
Parts:
- C41, C42: MPN (none) -> 100pF 50V C0G
- C43: MPN (none) -> 22uF 25V X7R
- C44, C49, C50: MPN (none) -> 100nF 50V X7R
- D10, D11, D12: MPN (none) -> 19-217/GHC-YR1S2/3T
- D5, D6, D7, D8, D9: MPN (none) -> KT-0603R
- LED1, LED2: MPN (none) -> SP420281N
- R40, R41, R42, R43, R53, R54: MPN (none) -> 10K 1%
- R44, R45: MPN (none) -> 220R 1%
- R46, R47: MPN (none) -> 6K8 1%
- RV1, RV2: MPN (none) -> 3386P-1-103TLF
- SW1, SW2, SW3, SW4, SW5: MPN (none) -> TS-1101-C-W
- U13: MPN (none) -> GN1640T
- U14, U15: MPN (none) -> 74LVC1G14GW,125
Changed lines of the file:
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@@
+      (effects (font (size 1.27 1.27)) hide)
+    )
+    (property "MPN" "TS-1101-C-W" (id 4) (at 182.88 97.79 0)
       (effects (font (size 1.27 1.27)) hide)
     )
@@
       (effects (font (size 1.27 1.27)) hide)
     )
+    (property "MPN" "10K 1%" (id 4) (at 209.55 44.45 0)
+      (effects (font (size 1.27 1.27)) hide)
+    )
     (pin "1")
     (pin "2")
@@
     )
     (property "Datasheet" "~" (id 3) (at 60.96 38.1 0)
+      (effects (font (size 1.27 1.27)) hide)
+    )
+    (property "MPN" "10K 1%" (id 4) (at 60.96 38.1 0)
       (effects (font (size 1.27 1.27)) hide)
     )
@@
       (effects (font (size 1.27 1.27)) hide)
     )
+    (property "MPN" "KT-0603R" (id 4) (at 137.16 149.86 0)
+      (effects (font (size 1.27 1.27)) hide)
+    )
     (pin "1")
     (pin "2")
@@
       (effects (font (size 1.27 1.27)) hide)
     )
+    (property "MPN" "19-217/GHC-YR1S2/3T" (id 4) (at 137.16 168.91 0)
+      (effects (font (size 1.27 1.27)) hide)
+    )
     (pin "1")
     (pin "2")
@@
       (effects (font (size 1.27 1.27)) hide)
     )
+    (property "MPN" "22uF 25V X7R" (id 4) (at 36.83 85.09 0)
+      (effects (font (size 1.27 1.27)) hide)
+    )
     (pin "1")
     (pin "2")
@@
     )
     (property "Datasheet" "~" (id 3) (at 209.55 53.34 0)
+      (effects (font (size 1.27 1.27)) hide)
+    )
+    (property "MPN" "6K8 1%" (id 4) (at 209.55 53.34 0)
       (effects (font (size 1.27 1.27)) hide)
     )
@@
       (effects (font (size 1.27 1.27)) hide)
     )
+    (property "MPN" "TS-1101-C-W" (id 4) (at 219.71 134.62 0)
+      (effects (font (size 1.27 1.27)) hide)
+    )
     (pin "1")
     (pin "2")
@@
       (effects (font (size 1.27 1.27)) hide)
     )
+    (property "MPN" "KT-0603R" (id 4) (at 137.16 143.51 0)
+      (effects (font (size 1.27 1.27)) hide)
+    )
     (pin "1")
     (pin "2")
@@
     )
     (property "Datasheet" "~" (id 3) (at 181.61 53.34 0)
+      (effects (font (size 1.27 1.27)) hide)
+    )
+    (property "MPN" "6K8 1%" (id 4) (at 181.61 53.34 0)
       (effects (font (size 1.27 1.27)) hide)
     )
@@
     )
     (property "Datasheet" "https://datasheet.lcsc.com/lcsc/1811041510_ARKLED-Wuxi-ARK-Tech-Elec-SP420281N_C122944.pdf" (id 3) (at 191.77 71.12 0)
+      (effects (font (size 1.27 1.27)) hide)
+    )
+    (property "MPN" "SP420281N" (id 4) (at 137.16 53.34 0)
       (effects (font (size 1.27 1.27)) hide)
     )
@@
     )
     (property "Datasheet" "" (id 3) (at 81.28 25.4 0)
+      (effects (font (size 1.27 1.27)) hide)
+    )
+    (property "MPN" "GN1640T" (id 4) (at 81.28 72.39 0)
       (effects (font (size 1.27 1.27)) hide)
     )
@@
       (effects (font (size 1.27 1.27)) hide)
     )
+    (property "MPN" "74LVC1G14GW,125" (id 4) (at 63.5 137.16 0)
+      (effects (font (size 1.27 1.27)) hide)
+    )
     (pin "1")
     (pin "2")
@@
       (effects (font (size 1.27 1.27)) hide)
     )
+    (property "MPN" "100nF 50V X7R" (id 4) (at 17.78 137.16 0)
+      (effects (font (size 1.27 1.27)) hide)
+    )
     (pin "1")
     (pin "2")
@@
     )
     (property "Datasheet" "https://datasheet.lcsc.com/lcsc/1811041510_ARKLED-Wuxi-ARK-Tech-Elec-SP420281N_C122944.pdf" (id 3) (at 191.77 113.03 0)
+      (effects (font (size 1.27 1.27)) hide)
+    )
+    (property "MPN" "SP420281N" (id 4) (at 137.16 95.25 0)
       (effects (font (size 1.27 1.27)) hide)
     )
@@
       (effects (font (size 1.27 1.27)) hide)
     )
+    (property "MPN" "KT-0603R" (id 4) (at 137.16 137.16 0)
+      (effects (font (size 1.27 1.27)) hide)
+    )
     (pin "1")
     (pin "2")
@@
     )
     (property "Datasheet" "~" (id 3) (at 48.26 143.51 0)
+      (effects (font (size 1.27 1.27)) hide)
+    )
+    (property "MPN" "10K 1%" (id 4) (at 48.26 143.51 0)
       (effects (font (size 1.27 1.27)) hide)
     )
@@
       (effects (font (size 1.27 1.27)) hide)
     )
+    (property "MPN" "TS-1101-C-W" (id 4) (at 182.88 134.62 0)
+      (effects (font (size 1.27 1.27)) hide)
+    )
     (pin "1")
     (pin "2")
@@
     )
     (property "Datasheet" "~" (id 3) (at 181.61 63.5 0)
+      (effects (font (size 1.27 1.27)) hide)
+    )
+    (property "MPN" "3386P-1-103TLF" (id 4) (at 181.61 63.5 0)
       (effects (font (size 1.27 1.27)) hide)
     )
@@
       (effects (font (size 1.27 1.27)) hide)
     )
+    (property "MPN" "220R 1%" (id 4) (at 38.1 46.99 0)
+      (effects (font (size 1.27 1.27)) hide)
+    )
     (pin "1")
     (pin "2")
@@
     )
     (property "Datasheet" "~" (id 3) (at 60.96 58.42 0)
+      (effects (font (size 1.27 1.27)) hide)
+    )
+    (property "MPN" "100pF 50V C0G" (id 4) (at 60.96 58.42 0)
       (effects (font (size 1.27 1.27)) hide)
     )
@@
       (effects (font (size 1.27 1.27)) hide)
     )
+    (property "MPN" "19-217/GHC-YR1S2/3T" (id 4) (at 137.16 156.21 0)
+      (effects (font (size 1.27 1.27)) hide)
+    )
     (pin "1")
     (pin "2")
@@
       (effects (font (size 1.27 1.27)) hide)
     )
+    (property "MPN" "74LVC1G14GW,125" (id 4) (at 63.5 168.91 0)
+      (effects (font (size 1.27 1.27)) hide)
+    )
     (pin "1")
     (pin "2")
@@
       (effects (font (size 1.27 1.27)) hide)
     )
+    (property "MPN" "19-217/GHC-YR1S2/3T" (id 4) (at 137.16 162.56 0)
+      (effects (font (size 1.27 1.27)) hide)
+    )
     (pin "1")
     (pin "2")
@@
       (effects (font (size 1.27 1.27)) hide)
     )
+    (property "MPN" "100nF 50V X7R" (id 4) (at 46.99 85.09 0)
+      (effects (font (size 1.27 1.27)) hide)
+    )
     (pin "1")
     (pin "2")
@@
     )
     (property "Datasheet" "~" (id 3) (at 181.61 44.45 0)
+      (effects (font (size 1.27 1.27)) hide)
+    )
+    (property "MPN" "10K 1%" (id 4) (at 181.61 44.45 0)
       (effects (font (size 1.27 1.27)) hide)
     )
@@
       (effects (font (size 1.27 1.27)) hide)
     )
+    (property "MPN" "3386P-1-103TLF" (id 4) (at 209.55 63.5 0)
+      (effects (font (size 1.27 1.27)) hide)
+    )
     (pin "1")
     (pin "2")
@@
     )
     (property "Datasheet" "~" (id 3) (at 48.26 175.26 0)
+      (effects (font (size 1.27 1.27)) hide)
+    )
+    (property "MPN" "10K 1%" (id 4) (at 48.26 175.26 0)
       (effects (font (size 1.27 1.27)) hide)
     )
@@
     )
     (property "Datasheet" "~" (id 3) (at 49.53 58.42 0)
+      (effects (font (size 1.27 1.27)) hide)
+    )
+    (property "MPN" "100pF 50V C0G" (id 4) (at 49.53 58.42 0)
       (effects (font (size 1.27 1.27)) hide)
     )
@@
       (effects (font (size 1.27 1.27)) hide)
     )
+    (property "MPN" "KT-0603R" (id 4) (at 137.16 130.81 0)
+      (effects (font (size 1.27 1.27)) hide)
+    )
     (pin "1")
     (pin "2")
@@
       (effects (font (size 1.27 1.27)) hide)
     )
+    (property "MPN" "TS-1101-C-W" (id 4) (at 257.81 97.79 0)
+      (effects (font (size 1.27 1.27)) hide)
+    )
     (pin "1")
     (pin "2")
@@
       (effects (font (size 1.27 1.27)) hide)
     )
+    (property "MPN" "KT-0603R" (id 4) (at 137.16 124.46 0)
+      (effects (font (size 1.27 1.27)) hide)
+    )
     (pin "1")
     (pin "2")
@@
     )
     (property "Datasheet" "~" (id 3) (at 49.53 38.1 0)
+      (effects (font (size 1.27 1.27)) hide)
+    )
+    (property "MPN" "10K 1%" (id 4) (at 49.53 38.1 0)
       (effects (font (size 1.27 1.27)) hide)
     )
@@
       (effects (font (size 1.27 1.27)) hide)
     )
+    (property "MPN" "220R 1%" (id 4) (at 38.1 49.53 0)
+      (effects (font (size 1.27 1.27)) hide)
+    )
     (pin "1")
     (pin "2")
@@
     )
     (property "Datasheet" "~" (id 3) (at 17.78 168.91 0)
+      (effects (font (size 1.27 1.27)) hide)
+    )
+    (property "MPN" "100nF 50V X7R" (id 4) (at 17.78 168.91 0)
       (effects (font (size 1.27 1.27)) hide)
     )
@@
       (effects (font (size 1.27 1.27)) hide)
     )
+    (property "MPN" "TS-1101-C-W" (id 4) (at 219.71 97.79 0)
+      (effects (font (size 1.27 1.27)) hide)
+    )

Commit message: Create IBOM, Add sheet info
Other:
- company: (none) -> Sleepy Pony Labs
- title: (none) -> Dual Rail Breadboard Power Supply
Changed lines of the file:
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@@
 (kicad_sch (version 20211123) (generator eeschema)
   (paper "A4")
+  (title_block
+    (title "Dual Rail Breadboard Power Supply")
+    (date "2023-06-11")
+    (rev "1")
+    (company "Sleepy Pony Labs")
+  )
   (junction (at 60.96 49.53) (diameter 0) (color 0 0 0 0)
   )
